File: hardware/hv_power_boost/hv_power_boost.kicad_sch (KiCad schematic)
At the start: 30 parts, among them J1 X6511WVS-02H-C60D48R1, J2 X6511WVS-03H-C60D48R1, Q1 FDS2734, U1 LM5155

Commit message: hardware(schematic): update hv boost board compensation value, update design document
Parts:
- removed C12: 0.47u/200V, Capacitor_SMD:C_1206_3216Metric, symbol Device:C_Small
- added R12: 150, Resistor_SMD:R_0603_1608Metric, symbol Device:R_Small
- C11: value 0.47u/200V -> 10u/400V; footprint Capacitor_SMD:C_1206_3216Metric -> (none); LCSC PN C725802 -> C46867081
- C6: value 18n -> 220n
- C7: value 33p -> 220p
- C8: value 1n -> 100n
- R10: value 50k -> 1M
- R11: value 300 -> 5.6k
- R5: value 30k -> 3.3k
- R7: value 0 -> 10
- R8: value 0 -> 100
- R9: value LMJ12MF1P0R047 -> WSLP1206R0330FEA; LCSC PN C5121701 -> C2084257
Connections:
- net GND: now also R12.2; no longer C13.2, R11.2
- new net: C13.2, R11.2, R12.1
