File: hardware/display_board_in4/display_board_in4.kicad_sch (KiCad schematic)
At the start: 164 parts, among them J1 CTRL, J2 HV_INPUT, J3 LED_CTRL, Q1 MMBTA42, Q10 MMBTA42, Q11 MMBTA42, Q12 MMBTA42, Q13 MMBTA42, Q14 MMBTA42, Q15 MMBTA42, Q16 MMBTA42, Q17 MMBTA42, Q18 MMBTA42, Q19 MMBTA42, Q2 MMBTA42, Q20 MMBTA42, Q21 MMBTA42, Q22 MMBTA42, Q23 MMBTA42, Q24 MMBTA42, Q25 MMBTA42, Q26 MMBTA42, Q27 MMBTA42, Q28 MMBTA42, Q29 MMBTA42, Q3 MMBTA42, Q30 MMBTA42, Q31 MMBTA42, Q32 MMBTA42, Q33 MMBTA42, Q34 MMBTA42, Q35 MMBTA42, Q36 MMBTA42, Q37 MMBTA42, Q38 MMBTA42, Q39 MMBTA42, Q4 MMBTA42, Q40 MMBTA42, Q41 MMBTA42, Q42 MMBTA42, Q43 MMBTA42, Q44 MMBTA42, Q45 MMBTA42, Q46 MMBTA42, Q47 MMBTA42, Q48 MMBTA42, Q49 MMBTA42, Q5 MMBTA42, Q50 MMBTA42, Q51 MMBTA42, Q52 MMBTA42, Q53 MMBTA42, Q54 MMBTA42, Q55 MMBTA42, Q56 MMBTA42, Q57 MMBTA42, Q58 MMBTA42, Q59 MMBTA42, Q6 MMBTA42, Q60 MMBTA42, Q7 MMBTA42, Q8 MMBTA42, Q9 MMBTA42, U1 PCA9685PW, U2 PCA9685PW, U3 PCA9685PW, U4 PCA9685PW

Commit message: hardware(schematic): update in4 display board current limit resistor to 68kOhm, update pin connector to 2X5 pin, no more GND1 needed, it's non-isloated
Parts:
- removed GND1: GND_TP, TestPoint:TestPoint_Pad_D2.0mm, symbol Connector:TestPoint_Small
- removed HV1: HV_TP, TestPoint:TestPoint_Pad_D2.0mm, symbol Connector:TestPoint_Small
- removed J1: CTRL, Connector_PinSocket_2.00mm:PinSocket_2x03_P2.00mm_Vertical, symbol Connector_Generic:Conn_02x03_Odd_Even
- removed J2: HV_INPUT, Connector_PinSocket_2.00mm:PinSocket_2x03_P2.00mm_Vertical, symbol Connector_Generic:Conn_02x03_Odd_Even
- removed J3: LED_CTRL, Connector_PinSocket_2.00mm:PinSocket_2x03_P2.00mm_Vertical, symbol Connector_Generic:Conn_02x03_Odd_Even
- removed SCL1: SCL_TP, TestPoint:TestPoint_Pad_D2.0mm, symbol Connector:TestPoint_Small
- removed SDA1: SDA_TP, TestPoint:TestPoint_Pad_D2.0mm, symbol Connector:TestPoint_Small
- added J2, J4: Conn_02x05_Counter_Clockwise, symbol Connector_Generic:Conn_02x05_Counter_Clockwise
- R1, R10, R11, R12, R13, R14, R15, R16, R17, R18, R19, R2, R20, R21, R22, R23, R24, R25, R26, R27, R28, R29, R3, R30, R31, R32, R33, R34, R35, R36, R37, R38, R39, R4, R40, R41, R42, R43, R44, R45, R46, R47, R48, R49, R5, R50, R51, R52, R53, R54, R55, R56, R57, R58, R59, R6, R60, R7, R8, R9: value 1.8k -> 68k; LCSC PN C1002 -> C23231
Connections:
- net GND1 is gone; now on net GND: GNDHV1.1, R1.1, R10.1, R11.1, R12.1, R13.1, R14.1, R15.1, R16.1, R17.1, R18.1, R19.1, R2.1, R20.1, R21.1, R22.1, R23.1, R24.1, R25.1, R26.1, R27.1, R28.1, R29.1, R3.1, R30.1, R31.1, R32.1, R33.1, R34.1, R35.1, R36.1, R37.1, R38.1, R39.1, R4.1, R40.1, R41.1, R42.1, R43.1, R44.1, R45.1, R46.1, R47.1, R48.1, R49.1, R5.1, R50.1, R51.1, R52.1, R53.1, R54.1, R55.1, R56.1, R57.1, R58.1, R59.1, R6.1, R60.1, R7.1, R8.1, R9.1
- net +3V3: now also J4.1 (Pin_1)
- net +5V: now also J4.6 (Pin_6)
- net DI: now also J4.3 (Pin_3)
- net GND: now also J2.10 (Pin_10), J2.8 (Pin_8), J2.9 (Pin_9), J4.4 (Pin_4), J4.5 (Pin_5), J4.7 (Pin_7), J4.8 (Pin_8)
- net N4_B0: now also U2.21 (LED14); no longer U3.6 (LED0)
- net N4_B1: now also U2.22 (LED15); no longer U3.7 (LED1)
- net N4_B2: now also U3.6 (LED0); no longer U3.8 (LED2)
- net N4_B3: now also U3.7 (LED1); no longer U3.9 (LED3)
- net N4_B4: now also U3.8 (LED2); no longer U3.10 (LED4)
- net N4_B5: now also U3.9 (LED3); no longer U3.11 (LED5)
- net N4_B6: now also U3.10 (LED4); no longer U3.12 (LED6)
- net N4_B7: now also U3.11 (LED5); no longer U3.13 (LED7)
- net N4_B8: now also U3.12 (LED6); no longer U3.15 (LED8)
- net N4_B9: now also U3.13 (LED7); no longer U3.16 (LED9)
- net N5_B0: now also U3.15 (LED8); no longer U3.17 (LED10)
- net N5_B1: now also U3.16 (LED9); no longer U3.18 (LED11)
- net N5_B2: now also U3.17 (LED10); no longer U3.19 (LED12)
- net N5_B3: now also U3.18 (LED11); no longer U3.20 (LED13)
- net N5_B4: now also U3.19 (LED12); no longer U3.21 (LED14)
- net N5_B5: now also U3.20 (LED13); no longer U3.22 (LED15)
- net N5_B6: now also U3.21 (LED14); no longer U4.6 (LED0)
- net N5_B7: now also U3.22 (LED15); no longer U4.7 (LED1)
- net N5_B8: now also U4.6 (LED0); no longer U4.8 (LED2)
- net N5_B9: now also U4.7 (LED1); no longer U4.9 (LED3)
- net N6_B0: now also U4.8 (LED2); no longer U4.10 (LED4)
- net N6_B1: now also U4.9 (LED3); no longer U4.11 (LED5)
- net N6_B2: now also U4.10 (LED4); no longer U4.12 (LED6)
- net N6_B3: now also U4.11 (LED5); no longer U4.13 (LED7)
- net N6_B4: now also U4.12 (LED6); no longer U4.15 (LED8)
- net N6_B5: now also U4.13 (LED7); no longer U4.16 (LED9)
- net N6_B6: now also U4.15 (LED8); no longer U4.17 (LED10)
- net N6_B7: now also U4.16 (LED9); no longer U4.18 (LED11)
- net N6_B8: now also U4.17 (LED10); no longer U4.19 (LED12)
- net N6_B9: now also U4.18 (LED11); no longer U4.20 (LED13)
- net SCL: now also J4.9 (Pin_9)
- net SDA: now also J4.10 (Pin_10)
- net ~{OE}: now also J4.2 (Pin_2)
- removed net ANODE: N1.A3 (A), N2.A3 (A), N3.A3 (A), N4.A3 (A), N5.A3 (A), N6.A3 (A)
- net DO: no longer names the net of D24.1 (DOUT)
- new net ANODE1: J2.1 (Pin_1), N1.A3 (A)
- new net ANODE2: J2.2 (Pin_2), N2.A3 (A)
- new net ANODE3: J2.3 (Pin_3), N3.A3 (A)
- new net ANODE4: J2.4 (Pin_4), N4.A3 (A)
- new net ANODE5: J2.5 (Pin_5), N5.A3 (A)
- new net ANODE6: J2.6 (Pin_6), N6.A3 (A)
- no-connect marks 4 -> 6
Other:
- note removed: "Operate BJT in saturartion mode Ie=(Vb-Vbe)/Re Ie=2.5mA=(3.3-0.9)/Re, Re=0.96kOhm"

Commit message: WIP(hardware): update in-4 display board
Parts:
- removed D1, D10, D11, D12, D13, D14, D15, D16, D17, D18, D19, D2, D20, D21, D22, D23, D24, D3, D4, D5, D6, D7, D8, D9: WS2812B-2020, LED_SMD:LED_WS2812B-2020_PLCC4_2.0x2.0mm, symbol LED:WS2812B-2020
- removed GNDHV1: GND_TP, TestPoint:TestPoint_Pad_D2.0mm, symbol Connector:TestPoint_Small
- added H1, H2, H3, H4: MountingHole, MountingHole:MountingHole_3.2mm_M3_DIN965, symbol Mechanical:MountingHole
- J1: renamed from J2; footprint (none) -> Connector_PinHeader_2.00mm:PinHeader_2x05_P2.00mm_Vertical_SMD
- J2: renamed from J4; footprint (none) -> Connector_PinHeader_2.00mm:PinHeader_2x05_P2.00mm_Vertical_SMD
- renumbered R61 to R1, R8 to R10, R9 to R11, R10 to R12, R11 to R13, R12 to R14, R13 to R15, R14 to R16, R15 to R17, R16 to R18, R17 to R19, R62 to R2, R18 to R20, R19 to R21, R20 to R22, R21 to R23, R22 to R24, R23 to R25, R24 to R26, R25 to R27, R26 to R28, R27 to R29, R1 to R3, R28 to R30, R29 to R31, R30 to R32, R31 to R33, R32 to R34, R33 to R35, R34 to R36, R35 to R37, R36 to R38, R37 to R39, R2 to R4, R38 to R40, R39 to R41, R40 to R42, R41 to R43, R42 to R44, R43 to R45, R44 to R46, R45 to R47, R46 to R48, R47 to R49, R3 to R5, R48 to R50, R49 to R51, R50 to R52, R51 to R53, R52 to R54, R53 to R55, R54 to R56, R55 to R57, R56 to R58, R57 to R59, R4 to R6, R58 to R60, R59 to R61, R60 to R62, R5 to R7, R6 to R8, R7 to R9
Connections:
- no-connect marks 6 -> 5
Other:
- added sheet LED_Backlight_Array (led_backlight_array.kicad_sch)

Commit message: WIP(hardware): in4 display board layout
Parts:
- removed J1, J2: Conn_02x05_Counter_Clockwise, Connector_PinHeader_2.00mm:PinHeader_2x05_P2.00mm_Vertical_SMD, symbol Connector_Generic:Conn_02x05_Counter_Clockwise
- added J1, J3: Conn_02x05_Odd_Even, Connector_PinSocket_2.00mm:PinSocket_2x05_P2.00mm_Vertical_SMD, symbol Connector_Generic:Conn_02x05_Odd_Even
Connections:
- net +3V3: now also J1.2 (Pin_2)
- net +5V: now also J1.9 (Pin_9)
- net ANODE1: now also J3.2 (Pin_2)
- net ANODE2: now also J3.4 (Pin_4)
- net ANODE3: now also J3.6 (Pin_6)
- net ANODE4: now also J3.8 (Pin_8)
- net ANODE5: now also J3.10 (Pin_10)
- net ANODE6: now also J3.9 (Pin_9)
- net DI: now also J1.6 (Pin_6)
- net GND: now also J1.10 (Pin_10), J1.5 (Pin_5), J1.7 (Pin_7), J1.8 (Pin_8), J3.1 (Pin_1), J3.3 (Pin_3), J3.5 (Pin_5)
- net SCL: now also J1.3 (Pin_3)
- net SDA: now also J1.1 (Pin_1)
- net ~{OE}: now also J1.4 (Pin_4)
Changed lines of the file:
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@@
 	)
 	(junction
+		(at 354.33 30.48)
+		(diameter 0)
+		(color 0 0 0 0)
+	)
+	(junction
 		(at 34.29 66.04)
 		(diameter 0)
@@
 	)
 	(junction
-		(at 354.33 27.94)
-		(diameter 0)
-		(color 0 0 0 0)
-	)
-	(junction
 		(at 34.29 76.2)
 		(diameter 0)
@@
 	)
 	(junction
+		(at 354.33 27.94)
+		(diameter 0)
+		(color 0 0 0 0)
+	)
+	(junction
 		(at 82.55 204.47)
 		(diameter 0)
@@
 	)
 	(junction
-		(at 354.33 30.48)
-		(diameter 0)
-		(color 0 0 0 0)
-	)
-	(junction
 		(at 241.3 265.43)
 		(diameter 0)
@@
 	(wire
 		(pts
-			(xy 354.33 27.94) (xy 354.33 30.48)
+			(xy 354.33 25.4) (xy 354.33 27.94)
 		)
 		(stroke
@@
 	(wire
 		(pts
+			(xy 354.33 27.94) (xy 354.33 30.48)
+		)
+		(stroke
+			(width 0)
+			(type default)
+		)
+	)
+	(wire
+		(pts
 			(xy 161.29 250.19) (xy 161.29 256.54)
 		)
@@
 	(wire
 		(pts
-			(xy 354.33 25.4) (xy 354.33 27.94)
-		)
-		(stroke
-			(width 0)
-			(type default)
-		)
-	)
-	(wire
-		(pts
 			(xy 107.95 59.69) (xy 107.95 73.66)
 		)
@@
 	)
 	(symbol
+		(lib_id "Connector_Generic:Conn_02x05_Odd_Even")
+		(at 388.62 31.75 0)
+		(mirror y)
+		(unit 1)
+		(exclude_from_sim no)
+		(in_bom yes)
+		(on_board yes)
+		(dnp no)
+		(property "Reference" "J1"
+			(at 387.35 20.32 0)
+			(effects
+				(font
+					(size 1.27 1.27)
+				)
+			)
+		)
+		(property "Value" "Conn_02x05_Odd_Even"
+			(at 387.35 22.86 0)
+			(effects
+				(font
+					(size 1.27 1.27)
+				)
+			)
+		)
+		(property "Footprint" "Connector_PinSocket_2.00mm:PinSocket_2x05_P2.00mm_Vertical_SMD"
+			(at 388.62 31.75 0)
+			(effects
+				(font
+					(size 1.27 1.27)
+				)
+				(hide yes)
+			)
+		)
+		(property "Datasheet" "~"
+			(at 388.62 31.75 0)
+			(effects
+				(font
+					(size 1.27 1.27)
+				)
+				(hide yes)
+			)
+		)
+		(property "Description" "Generic connector, double row, 02x05, odd/even pin numbering scheme (row 1 odd numbers, row 2 even numbers), script generated (kicad-library-utils/schlib/autogen/connector/)"
+			(at 388.62 31.75 0)
+			(effects
+				(font
+					(size 1.27 1.27)
+				)
+				(hide yes)
+			)
+		)
+		(pin "1"
+		)
+		(pin "3"
+		)
+		(pin "5"
+		)
+		(pin "7"
+		)
+		(pin "9"
+		)
+		(pin "2"
+		)
+		(pin "4"
+		)
+		(pin "6"
+		)
+		(pin "8"
+		)
+		(pin "10"
+		)
+		(instances
+			(project "display_board_in4"
+				(path "/4c618ed4-5bc0-4f4d-8f94-8dcddc8fa827"
+					(reference "J1")
+					(unit 1)
+				)
+			)
+		)
+	)
+	(symbol
 		(lib_id "power:GND1")
 		(at 55.88 266.7 0)
@@
 	)
 	(symbol
+		(lib_id "Connector_Generic:Conn_02x05_Odd_Even")
+		(at 349.25 30.48 0)
+		(mirror y)
+		(unit 1)
+		(exclude_from_sim no)
+		(in_bom yes)
+		(on_board yes)
+		(dnp no)
+		(property "Reference" "J3"
+			(at 347.98 19.05 0)
+			(effects
+				(font
+					(size 1.27 1.27)
+				)
+			)
+		)
+		(property "Value" "Conn_02x05_Odd_Even"
+			(at 347.98 21.59 0)
+			(effects
+				(font
+					(size 1.27 1.27)
+				)
+			)
+		)
+		(property "Footprint" "Connector_PinSocket_2.00mm:PinSocket_2x05_P2.00mm_Vertical_SMD"
+			(at 349.25 30.48 0)
+			(effects
+				(font
+					(size 1.27 1.27)
+				)
+				(hide yes)
+			)
+		)
+		(property "Datasheet" "~"
+			(at 349.25 30.48 0)
+			(effects
+				(font
+					(size 1.27 1.27)
+				)
+				(hide yes)
+			)
+		)
+		(property "Description" "Generic connector, double row, 02x05, odd/even pin numbering scheme (row 1 odd numbers, row 2 even numbers), script generated (kicad-library-utils/schlib/autogen/connector/)"
+			(at 349.25 30.48 0)
+			(effects
+				(font
+					(size 1.27 1.27)
+				)
+				(hide yes)
+			)
+		)
+		(pin "1"
+		)
+		(pin "3"
+		)
+		(pin "5"
+		)
+		(pin "7"
+		)
+		(pin "9"
+		)
+		(pin "2"
+		)
+		(pin "4"
+		)
+		(pin "6"
+		)
+		(pin "8"
+		)
+		(pin "10"
+		)
+		(instances
+			(project ""
+				(path "/4c618ed4-5bc0-4f4d-8f94-8dcddc8fa827"
+					(reference "J3")
+					(unit 1)
+				)
+			)
+		)
+	)
+	(symbol
 		(lib_id "Transistor_BJT:MMBTA42")
 		(at 237.49 193.04 0)
@@
 	)
 	(symbol
-		(lib_id "Connector_Generic:Conn_02x05_Counter_Clockwise")
-		(at 386.08 31.75 0)
-		(unit 1)
-		(exclude_from_sim no)
-		(in_bom yes)
-		(on_board yes)
-		(dnp no)
-		(fields_autoplaced yes)
-		(property "Reference" "J2"
-			(at 387.35 20.32 0)
-			(effects
-				(font
-					(size 1.27 1.27)
-				)
-			)
-		)
-		(property "Value" "Conn_02x05_Counter_Clockwise"
-			(at 387.35 22.86 0)
-			(effects
-				(font
-					(size 1.27 1.27)
-				)
-			)
-		)
-		(property "Footprint" "Connector_PinHeader_2.00mm:PinHeader_2x05_P2.00mm_Vertical_SMD"
-			(at 386.08 31.75 0)
-			(effects
-				(font
-					(size 1.27 1.27)
-				)
-				(hide yes)
-			)
-		)
-		(property "Datasheet" "~"
-			(at 386.08 31.75 0)
-			(effects
-				(font
-					(size 1.27 1.27)
-				)
-				(hide yes)
-			)
-		)
-		(property "Description" "Generic connector, double row, 02x05, counter clockwise pin numbering scheme (similar to DIP package numbering), script generated (kicad-library-utils/schlib/autogen/connector/)"
-			(at 386.08 31.75 0)
-			(effects
-				(font
-					(size 1.27 1.27)
-				)
-				(hide yes)
-			)
-		)
-		(pin "1"
-		)
-		(pin "4"
-		)
-		(pin "8"
-		)
-		(pin "9"
-		)
-		(pin "3"
-		)
-		(pin "7"
-		)
-		(pin "5"
-		)
-		(pin "10"
-		)
-		(pin "2"
-		)
-		(pin "6"
-		)
-		(instances
-			(project "display_board_in4"
-				(path "/4c618ed4-5bc0-4f4d-8f94-8dcddc8fa827"
-					(reference "J2")
-					(unit 1)
-				)
-			)
-		)
-	)
-	(symbol
 		(lib_id "Device:R_Small")
 		(at 236.22 259.08 180)
@@
 					(unit 1)
 				)
-			)
-		)
-	)
-	(symbol
-		(lib_id "Connector_Generic:Conn_02x05_Counter_Clockwise")
-		(at 346.71 30.48 0)
-		(unit 1)
-		(exclude_from_sim no)
-		(in_bom yes)
-		(on_board yes)
-		(dnp no)
-		(fields_autoplaced yes)
-		(property "Reference" "J1"
-			(at 347.98 19.05 0)
-			(effects
-				(font
-					(size 1.27 1.27)
-				)
-			)
-		)
-		(property "Value" "Conn_02x05_Counter_Clockwise"
-			(at 347.98 21.59 0)
-			(effects
-				(font
-					(size 1.27 1.27)
-				)
-			)
-		)
-		(property "Footprint" "Connector_PinHeader_2.00mm:PinHeader_2x05_P2.00mm_Vertical_SMD"
-			(at 346.71 30.48 0)
-			(effects
-				(font
-					(size 1.27 1.27)
-				)
-				(hide yes)
-			)
-		)
-		(property "Datasheet" "~"
-			(at 346.71 30.48 0)
-			(effects
-				(font
-					(size 1.27 1.27)
-				)
-				(hide yes)
-			)
-		)
-		(property "Description" "Generic connector, double row, 02x05, counter clockwise pin numbering scheme (similar to DIP package numbering), script generated (kicad-library-utils/schlib/autogen/connector/)"
-			(at 346.71 30.48 0)
-			(effects
-				(font
-					(size 1.27 1.27)
-				)
-				(hide yes)
-			)
-		)
-		(pin "1"
-		)
-		(pin "4"
-		)
-		(pin "8"
-		)
-		(pin "9"
-		)
-		(pin "3"
-		)
-		(pin "7"
-		)
-		(pin "5"
-		)
-		(pin "10"
-		)
-		(pin "2"
-		)
-		(pin "6"
-		)
-		(instances
-			(project ""
-				(path "/4c618ed4-5bc0-4f4d-8f94-8dcddc8fa827"
-					(reference "J1")
-					(unit 1)
-				)

Commit message: hardware(schematic): Update IN-4 schematic and layout
Parts:
- J1, J3: LCSC PN (none) -> C22373873
- R1, R2: LCSC PN C113303 -> C4190
Changed lines of the file:
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@@
 			)
 		)
+		(property "LCSC PN" "C22373873"
+			(at 388.62 31.75 0)
+			(effects
+				(font
+					(size 1.27 1.27)
+				)
+				(hide yes)
+			)
+		)
 		(pin "1"
 		)
@@
 			)
 		)
+		(property "LCSC PN" "C22373873"
+			(at 349.25 30.48 0)
+			(effects
+				(font
+					(size 1.27 1.27)
+				)
+				(hide yes)
+			)
+		)
 		(pin "1"
 		)
@@
 			)
 		)
-		(property "LCSC PN" "C113303"
+		(property "LCSC PN" "C4190"
 			(at 31.75 30.48 90)
 			(effects
@@
 			)
 		)
-		(property "LCSC PN" "C113303"
+		(property "LCSC PN" "C4190"
 			(at 29.21 30.48 90)
 			(effects

Commit message: hardware(display): add button and ALS sensor on display board, align the nixie tube
Parts:
- added C2: 1u, Capacitor_SMD:C_0603_1608Metric, symbol Device:C_Small
- added R63: 10k, Resistor_SMD:R_0402_1005Metric, symbol Device:R_Small
- added SW1: XKB5858-W-E-75, habonroof_kicad_library:XKB5858, symbol Johnson_Symbol_Lib:SW_push_RightAngle
- added U5: LTR-303ALS-01, OptoDevice:Lite-On_LTR-303ALS-01, symbol Sensor_Optical:LTR-303ALS-01
- R1, R2: now left out of the parts list
- R10, R11, R12, R13, R14, R15, R16, R17, R18, R19, R20, R21, R22, R23, R24, R25, R26, R27, R28, R29, R3, R30, R31, R32, R33, R34, R35, R36, R37, R38, R39, R4, R40, R41, R42, R43, R44, R45, R46, R47, R48, R49, R5, R50, R51, R52, R53, R54, R55, R56, R57, R58, R59, R6, R60, R61, R62, R7, R8, R9: value 68k -> 1k; LCSC PN C23231 -> C21190
Connections:
- net +3V3: now also C2.1, R63.1, U5.1 (VDD)
- net GND: now also C2.2, SW1.2, SW1.5, U5.3 (GND); no longer J1.5 (Pin_5), J1.7 (Pin_7), J1.8 (Pin_8)
- net SCL renamed I2C0_SCL
- net SDA renamed I2C0_SDA
- new net BTN_0: J1.8 (Pin_8), R63.2, SW1.4, SW1.6
- new net I2C1_SCL: J1.7 (Pin_7), U5.4 (SCL)
- new net I2C1_SDA: J1.5 (Pin_5), U5.6 (SDA)
- no-connect marks 5 -> 8
