File: hardware/display_board_in4/display_board_in4.kicad_sch (KiCad schematic)
At the start: 142 parts, among them J1 Conn_02x05_Odd_Even, J3 Conn_02x05_Odd_Even, Q1 MMBTA42, Q10 MMBTA42, Q11 MMBTA42, Q12 MMBTA42, Q13 MMBTA42, Q14 MMBTA42, Q15 MMBTA42, Q16 MMBTA42, Q17 MMBTA42, Q18 MMBTA42, Q19 MMBTA42, Q2 MMBTA42, Q20 MMBTA42, Q21 MMBTA42, Q22 MMBTA42, Q23 MMBTA42, Q24 MMBTA42, Q25 MMBTA42, Q26 MMBTA42, Q27 MMBTA42, Q28 MMBTA42, Q29 MMBTA42, Q3 MMBTA42, Q30 MMBTA42, Q31 MMBTA42, Q32 MMBTA42, Q33 MMBTA42, Q34 MMBTA42, Q35 MMBTA42, Q36 MMBTA42, Q37 MMBTA42, Q38 MMBTA42, Q39 MMBTA42, Q4 MMBTA42, Q40 MMBTA42, Q41 MMBTA42, Q42 MMBTA42, Q43 MMBTA42, Q44 MMBTA42, Q45 MMBTA42, Q46 MMBTA42, Q47 MMBTA42, Q48 MMBTA42, Q49 MMBTA42, Q5 MMBTA42, Q50 MMBTA42, Q51 MMBTA42, Q52 MMBTA42, Q53 MMBTA42, Q54 MMBTA42, Q55 MMBTA42, Q56 MMBTA42, Q57 MMBTA42, Q58 MMBTA42, Q59 MMBTA42, Q6 MMBTA42, Q60 MMBTA42, Q7 MMBTA42, Q8 MMBTA42, Q9 MMBTA42, U1 PCA9685PW, U2 PCA9685PW, U3 PCA9685PW, U4 PCA9685PW, U5 LTR-303ALS-01

Commit message: hw(display-in4): update LCSC PN and component status
Parts:
- C2: LCSC PN C5199872 -> C15849; now in the parts list
- J1, J3: now left out of the parts list
- R63: LCSC PN (none) -> C15402
- U5: now in the parts list
Changed lines of the file:
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@@
 		(unit 1)
 		(exclude_from_sim no)
-		(in_bom no)
+		(in_bom yes)
 		(on_board yes)
 		(dnp no)
@@
 			)
 		)
-		(property "LCSC PN" "C5199872"
+		(property "LCSC PN" "C15849"
 			(at 387.35 149.86 0)
 			(effects
@@
 		(unit 1)
 		(exclude_from_sim no)
-		(in_bom yes)
+		(in_bom no)
 		(on_board yes)
 		(dnp no)
@@
 		(unit 1)
 		(exclude_from_sim no)
-		(in_bom no)
+		(in_bom yes)
 		(on_board yes)
 		(dnp no)
@@
 		(unit 1)
 		(exclude_from_sim no)
-		(in_bom yes)
+		(in_bom no)
 		(on_board yes)
 		(dnp no)
@@
 			(at 341.63 60.96 0)
 			(effects
+				(font
+					(size 1.27 1.27)
+				)
+				(hide yes)
+			)
+		)
+		(property "LCSC PN" "C15402"
+			(at 341.63 60.96 0)
+			(effects

Commit message: chore(hw): add resistor LCSC PN
Parts:
- R63: LCSC PN C15402 -> C21189
- U5: LCSC PN (none) -> C364577
Changed lines of the file:
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@@
 			)
 		)
+		(property "LCSC PN" "C364577"
+			(at 361.95 149.86 0)
+			(effects
+				(font
+					(size 1.27 1.27)
+				)
+				(hide yes)
+			)
+		)
 		(pin "5"
 		)
@@
 			)
 		)
-		(property "LCSC PN" "C15402"
+		(property "LCSC PN" "C21189"
 			(at 341.63 60.96 0)
 			(effects
