File: hardware/display_board_in4/display_board_in4.kicad_pcb (KiCad board)
At the start: 4 copper layers, 230 x 50 mm, 191 parts, among them J1 Conn_02x05_Odd_Even, J3 Conn_02x05_Odd_Even, Q1 MMBTA42, Q10 MMBTA42, Q11 MMBTA42, Q12 MMBTA42, Q13 MMBTA42, Q14 MMBTA42, Q15 MMBTA42, Q16 MMBTA42, Q17 MMBTA42, Q18 MMBTA42, Q19 MMBTA42, Q2 MMBTA42, Q20 MMBTA42, Q21 MMBTA42, Q22 MMBTA42, Q23 MMBTA42, Q24 MMBTA42, Q25 MMBTA42, Q26 MMBTA42, Q27 MMBTA42, Q28 MMBTA42, Q29 MMBTA42, Q3 MMBTA42, Q30 MMBTA42, Q31 MMBTA42, Q32 MMBTA42, Q33 MMBTA42, Q34 MMBTA42, Q35 MMBTA42, Q36 MMBTA42, Q37 MMBTA42, Q38 MMBTA42, Q39 MMBTA42, Q4 MMBTA42, Q40 MMBTA42, Q41 MMBTA42, Q42 MMBTA42, Q43 MMBTA42, Q44 MMBTA42, Q45 MMBTA42, Q46 MMBTA42, Q47 MMBTA42, Q48 MMBTA42, Q49 MMBTA42, Q5 MMBTA42, Q50 MMBTA42, Q51 MMBTA42, Q52 MMBTA42, Q53 MMBTA42, Q54 MMBTA42, Q55 MMBTA42, Q56 MMBTA42, Q57 MMBTA42, Q58 MMBTA42, Q59 MMBTA42, Q6 MMBTA42, Q60 MMBTA42, Q7 MMBTA42, Q8 MMBTA42, Q9 MMBTA42, SW1 XKB5858-W-E-75, U1 PCA9685PW, U2 PCA9685PW, U3 PCA9685PW, U4 PCA9685PW, U5 LTR-303ALS-01

Commit message: WIP: schematic and layout
Parts:
- removed SW1: XKB5858-W-E-75, habonroof_kicad_library:XKB5858
- added R64: 0, Resistor_SMD:R_0603_1608Metric, B.Cu at (192.5, 130.6)
- R63: value 10k -> 0; footprint Resistor_SMD:R_0402_1005Metric -> Resistor_SMD:R_0603_1608Metric
- moved R63 11.0 mm to (196.3, 130.6), turned to 0 degrees
- turned N1 to 7.887 degrees
- turned N2 to 7.887 degrees
- turned N3 to 7.887 degrees
- turned N4 to 7.887 degrees
- turned N5 to 7.887 degrees
- turned N6 to 7.887 degrees
Connections:
- C2 pad 2: DISPLAY_TYPE -> GND
- D1 pad 2: DISPLAY_TYPE -> GND
- D10 pad 2: DISPLAY_TYPE -> GND
- D11 pad 2: DISPLAY_TYPE -> GND
- D12 pad 2: DISPLAY_TYPE -> GND
- D13 pad 2: DISPLAY_TYPE -> GND
- D14 pad 2: DISPLAY_TYPE -> GND
- D15 pad 2: DISPLAY_TYPE -> GND
- D16 pad 2: DISPLAY_TYPE -> GND
- D17 pad 2: DISPLAY_TYPE -> GND
- D18 pad 2: DISPLAY_TYPE -> GND
- D19 pad 2: DISPLAY_TYPE -> GND
- D2 pad 2: DISPLAY_TYPE -> GND
- D20 pad 2: DISPLAY_TYPE -> GND
- D21 pad 2: DISPLAY_TYPE -> GND
- D22 pad 2: DISPLAY_TYPE -> GND
- D23 pad 2: DISPLAY_TYPE -> GND
- D24 pad 2: DISPLAY_TYPE -> GND
- D25 pad 2: DISPLAY_TYPE -> GND
- D26 pad 2: DISPLAY_TYPE -> GND
- D27 pad 2: DISPLAY_TYPE -> GND
- D28 pad 2: DISPLAY_TYPE -> GND
- D29 pad 2: DISPLAY_TYPE -> GND
- D3 pad 2: DISPLAY_TYPE -> GND
- D30 pad 2: DISPLAY_TYPE -> GND
- D31 pad 2: DISPLAY_TYPE -> GND
- D32 pad 2: DISPLAY_TYPE -> GND
- D33 pad 2: DISPLAY_TYPE -> GND
- D34 pad 2: DISPLAY_TYPE -> GND
- D35 pad 2: DISPLAY_TYPE -> GND
- D36 pad 2: DISPLAY_TYPE -> GND
- D37 pad 2: DISPLAY_TYPE -> GND
- D38 pad 2: DISPLAY_TYPE -> GND
- D39 pad 2: DISPLAY_TYPE -> GND
- D4 pad 2: DISPLAY_TYPE -> GND
- D40 pad 2: DISPLAY_TYPE -> GND
- D41 pad 2: DISPLAY_TYPE -> GND
- D42 pad 2: DISPLAY_TYPE -> GND
- D43 pad 2: DISPLAY_TYPE -> GND
- D44 pad 2: DISPLAY_TYPE -> GND
- D45 pad 2: DISPLAY_TYPE -> GND
- D46 pad 2: DISPLAY_TYPE -> GND
- D47 pad 2: DISPLAY_TYPE -> GND
- D48 pad 2: DISPLAY_TYPE -> GND
- D5 pad 2: DISPLAY_TYPE -> GND
- D6 pad 2: DISPLAY_TYPE -> GND
- D7 pad 2: DISPLAY_TYPE -> GND
- D8 pad 2: DISPLAY_TYPE -> GND
- D9 pad 2: DISPLAY_TYPE -> GND
- J1 pad 10: DISPLAY_TYPE -> GND
- J1 pad 8: BTN_0 -> GND
- J3 pad 3: DISPLAY_TYPE -> GND
- J3 pad 5: DISPLAY_TYPE -> unconnected-(J3-Pin_5-Pad5)
- R10 pad 1: DISPLAY_TYPE -> GND
- R11 pad 1: DISPLAY_TYPE -> GND
- R12 pad 1: DISPLAY_TYPE -> GND
- R13 pad 1: DISPLAY_TYPE -> GND
- R14 pad 1: DISPLAY_TYPE -> GND
- R15 pad 1: DISPLAY_TYPE -> GND
- R16 pad 1: DISPLAY_TYPE -> GND
- R17 pad 1: DISPLAY_TYPE -> GND
- R18 pad 1: DISPLAY_TYPE -> GND
- R19 pad 1: DISPLAY_TYPE -> GND
- R20 pad 1: DISPLAY_TYPE -> GND
- R21 pad 1: DISPLAY_TYPE -> GND
- R22 pad 1: DISPLAY_TYPE -> GND
- R23 pad 1: DISPLAY_TYPE -> GND
- R24 pad 1: DISPLAY_TYPE -> GND
- R25 pad 1: DISPLAY_TYPE -> GND
- R26 pad 1: DISPLAY_TYPE -> GND
- R27 pad 1: DISPLAY_TYPE -> GND
- R28 pad 1: DISPLAY_TYPE -> GND
- R29 pad 1: DISPLAY_TYPE -> GND
- R3 pad 1: DISPLAY_TYPE -> GND
- R30 pad 1: DISPLAY_TYPE -> GND
- R31 pad 1: DISPLAY_TYPE -> GND
- R32 pad 1: DISPLAY_TYPE -> GND
- R33 pad 1: DISPLAY_TYPE -> GND
- R34 pad 1: DISPLAY_TYPE -> GND
- R35 pad 1: DISPLAY_TYPE -> GND
- R36 pad 1: DISPLAY_TYPE -> GND
- R37 pad 1: DISPLAY_TYPE -> GND
- R38 pad 1: DISPLAY_TYPE -> GND
- R39 pad 1: DISPLAY_TYPE -> GND
- R4 pad 1: DISPLAY_TYPE -> GND
- R40 pad 1: DISPLAY_TYPE -> GND
- R41 pad 1: DISPLAY_TYPE -> GND
- R42 pad 1: DISPLAY_TYPE -> GND
- R43 pad 1: DISPLAY_TYPE -> GND
- R44 pad 1: DISPLAY_TYPE -> GND
- R45 pad 1: DISPLAY_TYPE -> GND
- R46 pad 1: DISPLAY_TYPE -> GND
- R47 pad 1: DISPLAY_TYPE -> GND
- R48 pad 1: DISPLAY_TYPE -> GND
- R49 pad 1: DISPLAY_TYPE -> GND
- R5 pad 1: DISPLAY_TYPE -> GND
- R50 pad 1: DISPLAY_TYPE -> GND
- R51 pad 1: DISPLAY_TYPE -> GND
- R52 pad 1: DISPLAY_TYPE -> GND
- R53 pad 1: DISPLAY_TYPE -> GND
- R54 pad 1: DISPLAY_TYPE -> GND
- R55 pad 1: DISPLAY_TYPE -> GND
- R56 pad 1: DISPLAY_TYPE -> GND
- R57 pad 1: DISPLAY_TYPE -> GND
- R58 pad 1: DISPLAY_TYPE -> GND
- R59 pad 1: DISPLAY_TYPE -> GND
- R6 pad 1: DISPLAY_TYPE -> GND
- R60 pad 1: DISPLAY_TYPE -> GND
- R61 pad 1: DISPLAY_TYPE -> GND
- R62 pad 1: DISPLAY_TYPE -> GND
- R63 pad 1: +3V3 -> DISPLAY_TYPE
- R63 pad 2: BTN_0 -> GND
- R7 pad 1: DISPLAY_TYPE -> GND
- R8 pad 1: DISPLAY_TYPE -> GND
- R9 pad 1: DISPLAY_TYPE -> GND
- U1 pad 1: DISPLAY_TYPE -> GND
- U1 pad 14: DISPLAY_TYPE -> GND
- U1 pad 2: DISPLAY_TYPE -> GND
- U1 pad 24: DISPLAY_TYPE -> GND
- U1 pad 25: DISPLAY_TYPE -> GND
- U1 pad 3: DISPLAY_TYPE -> GND
- U1 pad 4: DISPLAY_TYPE -> GND
- U1 pad 5: DISPLAY_TYPE -> GND
- U2 pad 14: DISPLAY_TYPE -> GND
- U2 pad 2: DISPLAY_TYPE -> GND
- U2 pad 24: DISPLAY_TYPE -> GND
- U2 pad 25: DISPLAY_TYPE -> GND
- U2 pad 3: DISPLAY_TYPE -> GND
- U2 pad 4: DISPLAY_TYPE -> GND
- U2 pad 5: DISPLAY_TYPE -> GND
- U3 pad 1: DISPLAY_TYPE -> GND
- U3 pad 14: DISPLAY_TYPE -> GND
- U3 pad 24: DISPLAY_TYPE -> GND
- U3 pad 25: DISPLAY_TYPE -> GND
- U3 pad 3: DISPLAY_TYPE -> GND
- U3 pad 4: DISPLAY_TYPE -> GND
- U3 pad 5: DISPLAY_TYPE -> GND
- U4 pad 14: DISPLAY_TYPE -> GND
- U4 pad 24: DISPLAY_TYPE -> GND
- U4 pad 25: DISPLAY_TYPE -> GND
- U4 pad 3: DISPLAY_TYPE -> GND
- U4 pad 4: DISPLAY_TYPE -> GND
- U4 pad 5: DISPLAY_TYPE -> GND
- U5 pad 3: DISPLAY_TYPE -> GND
Routing:
- net GND: track 0.00 -> 267.8 mm, vias 0 -> 110
- net DISPLAY_TYPE: track 229.7 -> 23.5 mm, vias 110 -> 0
- net BTN_0: track 87.8 -> 0.00 mm, vias 1 -> 0
- net +3V3: track 200.0 -> 205.4 mm
- net /N1_D6: track 4.06 -> 5.39 mm
- net /N1_D3: track 5.52 -> 6.84 mm
- net /N1_D1: track 4.16 -> 5.46 mm
- net /N1_D2: track 4.83 -> 6.12 mm
- net /N1_D9: track 6.90 -> 8.12 mm
- net /N1_D8: track 4.33 -> 5.52 mm
- net /N1_D5: track 4.34 -> 5.50 mm
- net /N1_D0: track 4.35 -> 5.39 mm
- net /N1_D7: track 3.23 -> 4.19 mm
- net ANODE1: track 135.2 -> 134.3 mm
- added copper zone on B.Cu, net GND
- added copper zone on F.Cu, net GND
- added copper zone on In1.Cu, net GND
- added copper zone on In2.Cu, net GND
- removed copper zone on B.Cu, net DISPLAY_TYPE
- removed copper zone on F.Cu, net DISPLAY_TYPE
- removed copper zone on In1.Cu, net DISPLAY_TYPE
- removed copper zone on In2.Cu, net DISPLAY_TYPE

Commit message: WIP: hardware layout
Routing:
- net I2C1_SCL: track 61.8 -> 60.0 mm
- net /N2_D5: track 4.97 -> 6.47 mm
- net I2C1_SDA: track 65.9 -> 64.5 mm
- net /N2_D6: track 6.56 -> 7.89 mm
- net /N2_D2: track 6.50 -> 7.79 mm
- net /N3_D9: track 5.29 -> 6.51 mm
- net /N4_D1: track 3.98 -> 5.19 mm
- net /N2_D1: track 4.89 -> 6.10 mm
- net /N3_D3: track 4.75 -> 5.93 mm
- net /N3_D5: track 5.64 -> 6.79 mm
- net /N3_D1: track 4.82 -> 5.97 mm
- net /N2_D0: track 7.09 -> 8.13 mm
- net /N3_D0: track 4.14 -> 5.18 mm
- net /N3_D2: track 6.54 -> 7.55 mm
- net ANODE2: track 105.9 -> 105.0 mm
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
Commit message: hardware(in4): update in4 display board layout, fix the in4 rotation angle
Routing:
- net ANODE5: track 44.0 -> 41.3 mm
- net /N3_D8: track 3.53 -> 5.10 mm
- net /N4_D6: track 5.74 -> 7.25 mm
- net /N6_D8: track 4.69 -> 6.13 mm
- net /N6_D6: track 5.88 -> 7.22 mm
- net /N5_D6: track 4.82 -> 6.16 mm
- net /N4_D3: track 5.82 -> 7.15 mm
- net ANODE6: track 69.6 -> 70.9 mm
- net /N5_D2: track 5.69 -> 6.98 mm
- net /N4_D2: track 5.55 -> 6.85 mm
- net /N6_D2: track 5.13 -> 6.38 mm
- net /N6_D9: track 5.95 -> 7.17 mm
- net /N5_D9: track 5.64 -> 6.86 mm
- net /N2_D9: track 5.74 -> 6.96 mm
- net /N6_D1: track 4.91 -> 6.12 mm
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