File: hardware/main_board/hv_power_flyback.kicad_sch (KiCad schematic)
At the start: 28 parts, among them Q19 FDS2734, U8 LM5155

Commit message: hardware(sch): update anode mux resistor to reach 2.4mA for each tube, update 10kOhm PN
Parts:
- R77: LCSC PN C98220 -> C25804
Changed lines of the file:
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@@
 			)
 		)
-		(property "LCSC PN" "C98220"
+		(property "LCSC PN" "C25804"
 			(at 97.79 58.42 0)
 			(effects
