File: hardware/main_board/hv_power.kicad_sch (KiCad schematic)
At the start: 25 parts, among them Q3 FDS2734, U11 LM5155

Commit message: WIP: hardware layout
Parts:
- removed D6: ES5EB, Diode_SMD:D_SMB, symbol Device:D_Schottky
- removed R26: 10k, Resistor_SMD:R_0603_1608Metric, symbol Device:R_Small
- removed R32: 1M, Resistor_SMD:R_0603_1608Metric, symbol Device:R_Small
- added D4: STTH1R06B, Diode_SMD:D_SMB, symbol Device:D_Schottky
- added R80, R81: 499k, Resistor_SMD:R_0603_1608Metric, symbol Device:R_Small
- C26: renamed from C29; footprint Capacitor_SMD:C_0603_1608Metric -> Capacitor_SMD:C_0402_1005Metric; LCSC PN C519440 -> (none)
- C28: renamed from C30; footprint Capacitor_SMD:C_0603_1608Metric -> Capacitor_SMD:C_0402_1005Metric; LCSC PN C237177 -> (none)
- C29: renamed from C31; footprint Capacitor_SMD:C_0603_1608Metric -> Capacitor_SMD:C_0402_1005Metric; LCSC PN C576819 -> (none)
- C30: renamed from C32; footprint Capacitor_SMD:C_0603_1608Metric -> Capacitor_SMD:C_0402_1005Metric; LCSC PN C14663 -> (none)
- R69: renamed from R23; footprint Resistor_SMD:R_0603_1608Metric -> Resistor_SMD:R_0402_1005Metric; LCSC PN C304067 -> (none)
- R70: renamed from R24; footprint Resistor_SMD:R_0603_1608Metric -> Resistor_SMD:R_0402_1005Metric; LCSC PN C2828637 -> (none)
- R71: renamed from R25; footprint Resistor_SMD:R_0603_1608Metric -> Resistor_SMD:R_0402_1005Metric; LCSC PN C22961 -> (none)
- R74: renamed from R27; footprint Resistor_SMD:R_0603_1608Metric -> Resistor_SMD:R_0402_1005Metric; LCSC PN C114065 -> (none)
- R77: renamed from R29; footprint Resistor_SMD:R_0603_1608Metric -> Resistor_SMD:R_0402_1005Metric; LCSC PN C22859 -> (none)
- R78: renamed from R30; footprint Resistor_SMD:R_0603_1608Metric -> Resistor_SMD:R_0402_1005Metric; LCSC PN C22775 -> (none)
- renumbered C33 to C31, C34 to C33, C36 to C34, C37 to C35, L2 to L4, Q3 to Q20, R31 to R79, R33 to R82, R3 to R83, U11 to U15
Connections:
- net PWR_HV+: now also D4.1 (K), R80.1
- net at C35.1, R82.1, U15.8 (FB): now also R81.2
- net at L4.2, Q20.5 (D), Q20.6 (D)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: now also D4.2 (A)
- net PG: no longer names the net of U15.11 (PGOOD)
- net PWR_HV_VCC: no longer names the net of C31.2, U15.2 (VCC)
- new net: R80.2, R81.1
- no-connect marks 0 -> 1

Commit message: WIP: HV boost circuit integrate into main board
Parts:
- C34: footprint johnson:Cap_THT_D8.0mm_L12mm_Horizontal -> KiCad_Library:Cap_THT_D8.0mm_L12mm_Horizontal
- L4: footprint johnson:PowerInductor_8mmx8.5mm -> KiCad_Library:PowerInductor_8mmx8.5mm
Changed lines of the file:
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@@
 			)
 		)
-		(property "Footprint" "johnson:PowerInductor_8mmx8.5mm"
+		(property "Footprint" "KiCad_Library:PowerInductor_8mmx8.5mm"
 			(at 138.43 29.21 0)
 			(effects
@@
 			)
 		)
-		(property "Footprint" "johnson:Cap_THT_D8.0mm_L12mm_Horizontal"
+		(property "Footprint" "KiCad_Library:Cap_THT_D8.0mm_L12mm_Horizontal"
 			(at 210.82 44.45 0)
 			(effects
