File: hardware/main_board/hv_power.kicad_sch (KiCad schematic)
At the start: 25 parts, among them Q20 FDS2734, U15 LM5155

Commit message: WIP: Mainboard layout
Parts:
- removed C35: NC, Capacitor_SMD:C_0603_1608Metric, symbol Device:C_Small
- R77: value 10 -> 1
- R80, R81: footprint Resistor_SMD:R_0603_1608Metric -> Resistor_SMD:R_0402_1005Metric
- R82: footprint Resistor_SMD:R_0603_1608Metric -> Resistor_SMD:R_0402_1005Metric; LCSC PN C23189 -> (none)
- R83: footprint Resistor_SMD:R_0603_1608Metric -> Resistor_SMD:R_0402_1005Metric; LCSC PN C22808 -> (none)
Changed lines of the file:
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@@
-	)
-	(junction
-		(at 228.6 109.22)
-		(diameter 0)
-		(color 0 0 0 0)
 	)
 	(junction
@@
 	(wire
 		(pts
-			(xy 241.3 109.22) (xy 228.6 109.22)
-		)
-		(stroke
-			(width 0)
-			(type default)
-		)
-	)
-	(wire
-		(pts
 			(xy 166.37 35.56) (xy 166.37 38.1)
 		)
@@
 	(wire
 		(pts
-			(xy 228.6 90.17) (xy 241.3 90.17)
-		)
-		(stroke
-			(width 0)
-			(type default)
-		)
-	)
-	(wire
-		(pts
 			(xy 121.92 74.93) (xy 121.92 80.01)
 		)
@@
 	(wire
 		(pts
-			(xy 228.6 109.22) (xy 228.6 113.03)
-		)
-		(stroke
-			(width 0)
-			(type default)
-		)
-	)
-	(wire
-		(pts
 			(xy 104.14 80.01) (xy 111.76 80.01)
 		)
@@
 	(wire
 		(pts
-			(xy 241.3 97.79) (xy 241.3 109.22)
-		)
-		(stroke
-			(width 0)
-			(type default)
-		)
-	)
-	(wire
-		(pts
 			(xy 121.92 64.77) (xy 121.92 69.85)
 		)
@@
 	(wire
 		(pts
-			(xy 228.6 106.68) (xy 228.6 109.22)
+			(xy 228.6 106.68) (xy 228.6 113.03)
 		)
 		(stroke
@@
 		(pts
 			(xy 195.58 29.21) (xy 210.82 29.21)
-		)
-		(stroke
-			(width 0)
-			(type default)
-		)
-	)
-	(wire
-		(pts
-			(xy 241.3 92.71) (xy 241.3 90.17)
 		)
 		(stroke
@@
 			)
 		)
-		(property "Footprint" "Resistor_SMD:R_0603_1608Metric"
+		(property "Footprint" "Resistor_SMD:R_0402_1005Metric"
 			(at 228.6 68.58 0)
 			(effects
@@
 		)
 		(property "Description" "Resistor, small symbol"
+			(at 228.6 68.58 0)
+			(effects
+				(font
+					(size 1.27 1.27)
+				)
+				(hide yes)
+			)
+		)
+		(property "LCSC PN" ""
 			(at 228.6 68.58 0)
 			(effects
@@
 			)
 		)
-		(property "Value" "10"
+		(property "Value" "1"
 			(at 172.72 46.9899 0)
 			(effects
@@
 			)
 		)
-		(property "Footprint" "Resistor_SMD:R_0603_1608Metric"
+		(property "Footprint" "Resistor_SMD:R_0402_1005Metric"
 			(at 228.6 104.14 0)
 			(effects
@@
 			)
 		)
-		(property "LCSC PN" "C22808"
+		(property "LCSC PN" ""
 			(at 228.6 104.14 0)
 			(effects
@@
 			)
 		)
-		(property "Footprint" "Resistor_SMD:R_0603_1608Metric"
+		(property "Footprint" "Resistor_SMD:R_0402_1005Metric"
 			(at 228.6 95.25 0)
 			(effects
@@
 			)
 		)
-		(property "LCSC PN" "C23189"
+		(property "LCSC PN" ""
 			(at 228.6 95.25 0)
 			(effects
@@
 	)
 	(symbol
-		(lib_id "Device:C_Small")
-		(at 241.3 95.25 0)
-		(unit 1)
-		(exclude_from_sim yes)
-		(in_bom no)
-		(on_board yes)
-		(dnp yes)
-		(fields_autoplaced yes)
-		(property "Reference" "C35"
-			(at 243.84 93.9862 0)
-			(effects
-				(font
-					(size 1.27 1.27)
-				)
-				(justify left)
-			)
-		)
-		(property "Value" "NC"
-			(at 243.84 96.5262 0)
-			(effects
-				(font
-					(size 1.27 1.27)
-				)
-				(justify left)
-			)
-		)
-		(property "Footprint" "Capacitor_SMD:C_0603_1608Metric"
-			(at 241.3 95.25 0)
-			(effects
-				(font
-					(size 1.27 1.27)
-				)
-				(hide yes)
-			)
-		)
-		(property "Datasheet" "~"
-			(at 241.3 95.25 0)
-			(effects
-				(font
-					(size 1.27 1.27)
-				)
-				(hide yes)
-			)
-		)
-		(property "Description" "Unpolarized capacitor, small symbol"
-			(at 241.3 95.25 0)
-			(effects
-				(font
-					(size 1.27 1.27)
-				)
-				(hide yes)
-			)
-		)
-		(property "LCSC PN" ""
-			(at 241.3 95.25 0)
-			(effects
-				(font
-					(size 1.27 1.27)
-				)
-				(hide yes)
-			)
-		)
-		(pin "2"
-		)
-		(pin "1"
-		)
-		(instances
-			(project "main_board"
-				(path "/62950e93-3f98-4dee-9256-8213caa98ee7/529bf63b-1ea4-4ef4-8d8a-4c1847b02979"
-					(reference "C35")
-					(unit 1)
-				)
-			)
-		)
-	)
-	(symbol
 		(lib_id "Device:R_Small")
 		(at 228.6 57.15 0)
@@
 			)
 		)
-		(property "Footprint" "Resistor_SMD:R_0603_1608Metric"
+		(property "Footprint" "Resistor_SMD:R_0402_1005Metric"
 			(at 228.6 57.15 0)
 			(effects
@@
 			(at 228.6 57.15 0)
 			(effects
+				(font
+					(size 1.27 1.27)
+				)
+				(hide yes)
+			)
+		)
+		(property "LCSC PN" ""
+			(at 228.6 57.15 0)
+			(effects

Commit message: WIP: update mainboard componemt LCSC PN
Parts:
- C28: value 120n -> 220n
- C29: value 50p -> 220p
- C30: LCSC PN (none) -> C1525
- C34: now not fitted
- R74: value 22k -> 3.3k
Changed lines of the file:
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@@
 		(in_bom yes)
 		(on_board yes)
-		(dnp no)
+		(dnp yes)
 		(fields_autoplaced yes)
 		(property "Reference" "C34"
@@
 			)
 		)
-		(property "Value" "22k"
+		(property "Value" "3.3k"
 			(at 114.3 69.8499 0)
 			(effects
@@
 			)
 		)
-		(property "Value" "50p"
+		(property "Value" "220p"
 			(at 124.46 73.6662 0)
 			(effects
@@
 			)
 		)
-		(property "LCSC PN" ""
+		(property "LCSC PN" "C1525"
 			(at 165.1 60.96 0)
 			(effects
@@
 			)
 		)
-		(property "Value" "120n"
+		(property "Value" "220n"
 			(at 114.3 76.2062 0)
 			(effects

Commit message: WIP: update component LCSCPN
Parts:
- C26: LCSC PN (none) -> C309457
- C28: LCSC PN (none) -> C16772
- C29: LCSC PN (none) -> C1530
- R69: LCSC PN (none) -> C166559
- R70: LCSC PN (none) -> C2766803
- R71: LCSC PN (none) -> C25546
- R74: LCSC PN (none) -> C25890
- R77: LCSC PN (none) -> C25086
- R78: LCSC PN (none) -> C25076
- R80, R81: LCSC PN (none) -> C25793
- R82: LCSC PN (none) -> C881140
- R83: LCSC PN (none) -> C25082
Changed lines of the file:
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@@
 			)
 		)
-		(property "LCSC PN" ""
+		(property "LCSC PN" "C25793"
 			(at 228.6 68.58 0)
 			(effects
@@
 			)
 		)
-		(property "LCSC PN" ""
+		(property "LCSC PN" "C25086"
 			(at 170.18 45.72 0)
 			(effects
@@
 			)
 		)
-		(property "LCSC PN" ""
+		(property "LCSC PN" "C2766803"
 			(at 92.71 53.34 0)
 			(effects
@@
 			)
 		)
-		(property "LCSC PN" ""
+		(property "LCSC PN" "C25082"
 			(at 228.6 104.14 0)
 			(effects
@@
 			)
 		)
-		(property "LCSC PN" ""
+		(property "LCSC PN" "C166559"
 			(at 92.71 35.56 0)
 			(effects
@@
 			)
 		)
-		(property "LCSC PN" ""
+		(property "LCSC PN" "C25890"
 			(at 111.76 68.58 0)
 			(effects
@@
 			)
 		)
-		(property "LCSC PN" ""
+		(property "LCSC PN" "C25076"
 			(at 171.45 57.15 0)
 			(effects
@@
 			)
 		)
-		(property "LCSC PN" ""
+		(property "LCSC PN" "C881140"
 			(at 228.6 95.25 0)
 			(effects
@@
 			)
 		)
-		(property "LCSC PN" ""
+		(property "LCSC PN" "C309457"
 			(at 104.14 71.12 0)
 			(effects
@@
 			)
 		)
-		(property "LCSC PN" ""
+		(property "LCSC PN" "C25546"
 			(at 96.52 66.04 0)
 			(effects
@@
 			)
 		)
-		(property "LCSC PN" ""
+		(property "LCSC PN" "C25793"
 			(at 228.6 57.15 0)
 			(effects
@@
 			)
 		)
-		(property "LCSC PN" ""
+		(property "LCSC PN" "C1530"
 			(at 121.92 72.39 0)
 			(effects
@@
 			)
 		)
-		(property "LCSC PN" ""
+		(property "LCSC PN" "C16772"
 			(at 111.76 74.93 0)
 			(effects

Commit message: hw(main_board): update LCSC PN
Parts:
- C25: value 100u -> 10u; footprint Capacitor_SMD:C_1206_3216Metric -> Capacitor_SMD:C_0805_2012Metric; LCSC PN C15008 -> C6119932
Changed lines of the file:
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@@
 			)
 		)
-		(property "Value" "100u"
+		(property "Value" "10u"
 			(at 63.5 55.8862 0)
 			(effects
@@
 			)
 		)
-		(property "Footprint" "Capacitor_SMD:C_1206_3216Metric"
+		(property "Footprint" "Capacitor_SMD:C_0805_2012Metric"
 			(at 60.96 54.61 0)
 			(effects
@@
 			)
 		)
-		(property "LCSC PN" "C15008"
+		(property "LCSC PN" "C6119932"
 			(at 60.96 54.61 0)
 			(effects
