File: hardware/main_board/nixie_anode_mux.kicad_sch (KiCad schematic)
At the start: 38 parts, among them Q10 MMBTA42, Q11 MMBTA92, Q12 MMBTA42, Q13 MMBTA92, Q14 MMBTA42, Q15 MMBTA92, Q4 MMBTA92, Q5 MMBTA42, Q6 MMBTA42, Q7 MMBTA92, Q8 MMBTA42, Q9 MMBTA92, U13 74HC238

Commit message: hardware(sch): update anode mux resistor to reach 2.4mA for each tube, update 10kOhm PN
Parts:
- R35, R40, R44, R48, R51, R52: value 47k -> 9.1k; LCSC PN C25792 -> C23260
Changed lines of the file:
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@@
 			)
 		)
-		(property "Value" "47k"
+		(property "Value" "9.1k"
 			(at 68.58 102.87 90)
 			(effects
@@
 			)
 		)
-		(property "LCSC PN" "C25792"
+		(property "LCSC PN" "C23260"
 			(at 68.58 105.41 90)
 			(effects
@@
 			)
 		)
-		(property "Value" "47k"
+		(property "Value" "9.1k"
 			(at 132.08 46.99 90)
 			(effects
@@
 			)
 		)
-		(property "LCSC PN" "C25792"
+		(property "LCSC PN" "C23260"
 			(at 132.08 49.53 90)
 			(effects
@@
 			)
 		)
-		(property "Value" "47k"
+		(property "Value" "9.1k"
 			(at 201.93 104.14 90)
 			(effects
@@
 			)
 		)
-		(property "LCSC PN" "C25792"
+		(property "LCSC PN" "C23260"
 			(at 201.93 106.68 90)
 			(effects
@@
 			)
 		)
-		(property "Value" "47k"
+		(property "Value" "9.1k"
 			(at 196.85 48.26 90)
 			(effects
@@
 			)
 		)
-		(property "LCSC PN" "C25792"
+		(property "LCSC PN" "C23260"
 			(at 196.85 50.8 90)
 			(effects
@@
 			)
 		)
-		(property "Value" "47k"
+		(property "Value" "9.1k"
 			(at 133.35 102.87 90)
 			(effects
@@
 			)
 		)
-		(property "LCSC PN" "C25792"
+		(property "LCSC PN" "C23260"
 			(at 133.35 105.41 90)
 			(effects
@@
 			)
 		)
-		(property "Value" "47k"
+		(property "Value" "9.1k"
 			(at 68.58 46.99 90)
 			(effects
@@
 			)
 		)
-		(property "LCSC PN" "C25792"
+		(property "LCSC PN" "C23260"
 			(at 68.58 49.53 90)
 			(effects

Commit message: WIP: schematic and layout
Parts:
- added Q16, Q19: MMBTA92, Package_TO_SOT_SMD:SOT-23, symbol Transistor_BJT:MMBTA92
- added Q18, Q3: MMBTA42, Package_TO_SOT_SMD:SOT-23, symbol Transistor_BJT:MMBTA42
- added R13, R56: 470k, Resistor_SMD:R_0402_1005Metric, symbol Device:R_Small
- added R14, R58: 1M, Resistor_SMD:R_0402_1005Metric, symbol Device:R_Small
- added R3, R55: 10k, Resistor_SMD:R_0402_1005Metric, symbol Device:R_Small
- added R54, R60: 9.1k, Resistor_SMD:R_0402_1005Metric, symbol Device:R_Small
Connections:
- net GND: now also Q18.2 (E), Q3.2 (E)
- net HV_POWER: now also Q16.2 (E), Q19.2 (E)
- net T7_B: now reaches U13.7 (Y7)
- net T7_B: now also R55.1
- net T6_B: now reaches U13.9 (Y6)
- net T6_B: now also R3.1
- new net: Q18.1 (B), R55.2
- new net: Q19.3 (C), R56.2, R58.2, R60.1
- new net: Q19.1 (B), R58.1
- new net: Q3.3 (C), R13.1
- new net: Q16.3 (C), R13.2, R14.2, R54.1
- new net: Q3.1 (B), R3.2
- new net: Q18.3 (C), R56.1
- new net: Q16.1 (B), R14.1
- new net T6_E: R54.2
- new net T7_E: R60.2
- no-connect marks 2 -> 0
Other:
- moved on the sheet: Q10, Q11, Q12, Q13, Q14, Q15, R30, R31, R32, R41, R42, R45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

Commit message: WIP: hardware layout
Parts:
- renumbered C41 to C24, Q7 to Q10, Q15 to Q11, Q3 to Q12, Q8 to Q13, Q16 to Q14, Q9 to Q15, Q10 to Q16, Q18 to Q17, Q11 to Q18, Q5 to Q4, Q12 to Q5, Q4 to Q6, Q13 to Q7, Q6 to Q8, Q14 to Q9, R36 to R37, R31 to R38, R34 to R39, R42 to R40, R21 to R41, R49 to R42, R35 to R43, R51 to R44, R46 to R45, R32 to R46, R37 to R47, R41 to R48, R39 to R49, R47 to R50, R40 to R51, R48 to R52, R3 to R53, R33 to R54, R13 to R55, R38 to R56, R14 to R57, R43 to R58, R54 to R59, R44 to R60, R30 to R61, R55 to R62, R45 to R63, R56 to R64, R50 to R65, R58 to R66, R52 to R67, R60 to R68, U13 to U14

Commit message: WIP: mainboard schematic
Parts:
- R43, R44, R51, R52, R59, R60, R67, R68: LCSC PN C23260 -> C4968
Changed lines of the file:
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@@
 			)
 		)
-		(property "LCSC PN" "C23260"
+		(property "LCSC PN" "C4968"
 			(at 264.16 113.03 90)
 			(effects
@@
 			)
 		)
-		(property "LCSC PN" "C23260"
+		(property "LCSC PN" "C4968"
 			(at 262.89 50.8 90)
 			(effects
@@
 			)
 		)
-		(property "LCSC PN" "C23260"
+		(property "LCSC PN" "C4968"
 			(at 132.08 49.53 90)
 			(effects
@@
 			)
 		)
-		(property "LCSC PN" "C23260"
+		(property "LCSC PN" "C4968"
 			(at 137.16 109.22 90)
 			(effects
@@
 			)
 		)
-		(property "LCSC PN" "C23260"
+		(property "LCSC PN" "C4968"
 			(at 196.85 50.8 90)
 			(effects
@@
 			)
 		)
-		(property "LCSC PN" "C23260"
+		(property "LCSC PN" "C4968"
 			(at 68.58 107.95 90)
 			(effects
@@
 			)
 		)
-		(property "LCSC PN" "C23260"
+		(property "LCSC PN" "C4968"
 			(at 195.58 111.76 90)
 			(effects
@@
 			)
 		)
-		(property "LCSC PN" "C23260"
+		(property "LCSC PN" "C4968"
 			(at 68.58 49.53 90)
 			(effects
