File: hardware/main_board/nixie_anode_mux.kicad_sch (KiCad schematic)
At the start: 50 parts, among them Q10 MMBTA92, Q11 MMBTA92, Q12 MMBTA42, Q13 MMBTA42, Q14 MMBTA92, Q15 MMBTA92, Q16 MMBTA42, Q17 MMBTA42, Q18 MMBTA92, Q19 MMBTA92, Q4 MMBTA42, Q5 MMBTA42, Q6 MMBTA92, Q7 MMBTA92, Q8 MMBTA42, Q9 MMBTA42, U14 74HC238

Commit message: hw(main_board): update LCSC PN
Parts:
- R39, R40, R47, R48, R55, R56, R63, R64: LCSC PN C25790 -> C100446
- R43, R44, R51, R52, R59, R60, R67, R68: LCSC PN C4968 -> C100555
Changed lines of the file:
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@@
 			)
 		)
-		(property "LCSC PN" "C4968"
+		(property "LCSC PN" "C100555"
 			(at 264.16 113.03 90)
 			(effects
@@
 			)
 		)
-		(property "LCSC PN" "C25790"
+		(property "LCSC PN" "C100446"
 			(at 114.3 109.22 90)
 			(effects
@@
 			)
 		)
-		(property "LCSC PN" "C25790"
+		(property "LCSC PN" "C100446"
 			(at 173.99 50.8 90)
 			(effects
@@
 			)
 		)
-		(property "LCSC PN" "C4968"
+		(property "LCSC PN" "C100555"
 			(at 262.89 50.8 90)
 			(effects
@@
 			)
 		)
-		(property "LCSC PN" "C25790"
+		(property "LCSC PN" "C100446"
 			(at 109.22 49.53 90)
 			(effects
@@
 			)
 		)
-		(property "LCSC PN" "C4968"
+		(property "LCSC PN" "C100555"
 			(at 132.08 49.53 90)
 			(effects
@@
 			)
 		)
-		(property "LCSC PN" "C25790"
+		(property "LCSC PN" "C100446"
 			(at 172.72 111.76 90)
 			(effects
@@
 			)
 		)
-		(property "LCSC PN" "C25790"
+		(property "LCSC PN" "C100446"
 			(at 240.03 50.8 90)
 			(effects
@@
 			)
 		)
-		(property "LCSC PN" "C4968"
+		(property "LCSC PN" "C100555"
 			(at 137.16 109.22 90)
 			(effects
@@
 			)
 		)
-		(property "LCSC PN" "C4968"
+		(property "LCSC PN" "C100555"
 			(at 196.85 50.8 90)
 			(effects
@@
 			)
 		)
-		(property "LCSC PN" "C25790"
+		(property "LCSC PN" "C100446"
 			(at 241.3 113.03 90)
 			(effects
@@
 			)
 		)
-		(property "LCSC PN" "C25790"
+		(property "LCSC PN" "C100446"
 			(at 45.72 49.53 90)
 			(effects
@@
 			)
 		)
-		(property "LCSC PN" "C4968"
+		(property "LCSC PN" "C100555"
 			(at 68.58 107.95 90)
 			(effects
@@
 			)
 		)
-		(property "LCSC PN" "C25790"
+		(property "LCSC PN" "C100446"
 			(at 45.72 107.95 90)
 			(effects
@@
 			)
 		)
-		(property "LCSC PN" "C4968"
+		(property "LCSC PN" "C100555"
 			(at 195.58 111.76 90)
 			(effects
@@
 			)
 		)
-		(property "LCSC PN" "C4968"
+		(property "LCSC PN" "C100555"
 			(at 68.58 49.53 90)
 			(effects

Commit message: fix(hw): fix BQ25601 can not set 12V OVP after power reset. Due to BQ25601 will reset the register after power reset, HUSB238 need to ask 5V for the first stage, then use I2C to ask 12V PDO to makes the HV boost converter for better efficiency.
Connections:
- net +5V renamed +3V3
Changed lines of the file:
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@@
 			)
 		)
-		(property "Value" "+5V"
-			(at 90.17 135.89 0)
+		(property "Value" "+3V3"
+			(at 92.71 139.6999 0)
 			(effects
 				(font
 					(size 1.27 1.27)
 				)
+				(justify left)
 			)
 		)
