File: hardware/main_board/gasgauge.kicad_sch (KiCad schematic)
At the start: 6 parts, among them U16 BQ27441DRZR-G1A

Commit message: WIP: hardware layout
Parts:
- renumbered C12 to C27, C15 to C32, R22 to R72, R15 to R75, R19 to R76
Changed lines of the file:
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@@
 		(dnp no)
 		(fields_autoplaced yes)
-		(property "Reference" "R15"
+		(property "Reference" "R75"
 			(at 120.65 95.25 0)
 			(effects
@@
 			(project "main_board"
 				(path "/62950e93-3f98-4dee-9256-8213caa98ee7/23960838-3dbf-4684-acd4-edccf335cc3f"
-					(reference "R15")
+					(reference "R75")
 					(unit 1)
 				)
@@
 		(dnp no)
 		(fields_autoplaced yes)
-		(property "Reference" "R22"
+		(property "Reference" "R72"
 			(at 96.52 72.39 90)
 			(effects
@@
 			(project "main_board"
 				(path "/62950e93-3f98-4dee-9256-8213caa98ee7/23960838-3dbf-4684-acd4-edccf335cc3f"
-					(reference "R22")
+					(reference "R72")
 					(unit 1)
 				)
@@
 		(on_board yes)
 		(dnp no)
-		(property "Reference" "C15"
+		(property "Reference" "C32"
 			(at 177.546 86.106 0)
 			(effects
@@
 			(project "main_board"
 				(path "/62950e93-3f98-4dee-9256-8213caa98ee7/23960838-3dbf-4684-acd4-edccf335cc3f"
-					(reference "C15")
+					(reference "C32")
 					(unit 1)
 				)
@@
 		(dnp no)
 		(fields_autoplaced yes)
-		(property "Reference" "C12"
+		(property "Reference" "C27"
 			(at 107.95 90.1762 0)
 			(effects
@@
 			(project "main_board"
 				(path "/62950e93-3f98-4dee-9256-8213caa98ee7/23960838-3dbf-4684-acd4-edccf335cc3f"
-					(reference "C12")
+					(reference "C27")
 					(unit 1)
 				)
@@
 		(dnp no)
 		(fields_autoplaced yes)
-		(property "Reference" "R19"
+		(property "Reference" "R76"
 			(at 162.56 77.47 0)
 			(effects
@@
 			(project "main_board"
 				(path "/62950e93-3f98-4dee-9256-8213caa98ee7/23960838-3dbf-4684-acd4-edccf335cc3f"
-					(reference "R19")
+					(reference "R76")
 					(unit 1)
 				)

Commit message: fix(hw): fix BQ25601 can not set 12V OVP after power reset. Due to BQ25601 will reset the register after power reset, HUSB238 need to ask 5V for the first stage, then use I2C to ask 12V PDO to makes the HV boost converter for better efficiency.
Parts:
- C27: value 100n -> 1u; LCSC PN C1525 -> (none)
Changed lines of the file:
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@@
 			)
 		)
-		(property "Value" "100n"
+		(property "Value" "1u"
 			(at 107.95 92.7162 0)
 			(effects
@@
 			)
 		)
-		(property "LCSC PN" "C1525"
+		(property "LCSC PN" ""
 			(at 105.41 91.44 0)
 			(effects
