File: hardware/main_board/main_board.kicad_sch (KiCad schematic)
At the start: 98 parts, among them J1 USB_C_Receptacle_USB2.0_16P, J2 BAT1, J3 Conn_02x05_Odd_Even, J4 Conn_02x05_Odd_Even, Q1 FDMC4435BZ, Q2 MMBT3904, Q3 MMBT3904, SW1 PTS645VK31LFS, SW2 PTS645VK31LFS, SW3 PTS645VK31LFS, U1 SRV05-4, U10 TPS61022, U11 ESP32-S3-WROOM1, U12 TPS2121, U13 TPS22810DBVR, U2 CP2102N-A02-GQFN28, U3 HUSB238_002DD, U4 TPS22918DBVR, U5 BQ25601, U6 DFPlayer_mini, U7 DS3231MZ, U8 TPS63802, U9 NCH2800HV

Commit message: fix(hw): fix BQ25601 can not set 12V OVP after power reset. Due to BQ25601 will reset the register after power reset, HUSB238 need to ask 5V for the first stage, then use I2C to ask 12V PDO to makes the HV boost converter for better efficiency.
Parts:
- added D5: SMF28A, Diode_SMD:D_SMF, symbol Diode:SMF28A
- R20, R21: value 4.7k -> 1.3k
- R22, R23: value 4.7k -> 1.3k; LCSC PN C25900 -> C881388
- R8: value 10k -> 0; LCSC PN C25744 -> C17168
Connections:
- net +3V3: now also R84.2
- net +5V: no longer R84.2
- net HV_PWR+: now also U13.6 (VOUT); no longer U13.4 (VOUT)
- net I2C0_SCL: now also U3.6 (SDA)
- net I2C0_SDA: now also U3.7 (SCL)
- net PGND1: now also D5.2 (A2)
- net VBUS: now also Q1.1 (S); no longer Q1.5 (D)
- net at U4.4 (CT): now also C7.1; no longer U6.1 (Vcc)
- net at U4.6 (VOUT): now also U6.1 (Vcc); no longer C7.1
- net at C3.1, J1.A4 (VBUS), J1.A9 (VBUS)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: now also Q1.5 (D), D5.1 (A1); no longer Q1.1 (S), U1.5 (VP)
- net at C23.1: now also U13.4 (CT); no longer U13.6 (CT)
- no-connect marks 46 -> 45
Other:
- note added: "I2C address: 0x08"
- moved on the sheet: Q1
Changed lines of the file:
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@@
 		)
 	)
+	(text "I2C address: 0x08"
+		(exclude_from_sim no)
+		(at 103.632 72.898 0)
+		(effects
+			(font
+				(size 1.27 1.27)
+			)
+		)
+	)
 	(text "RVSET(kΩ) - VSET\n0     - 5\n6.04  - 9\n10    - 12\n14    - 15\n17.8  - 18\nOpen  - 20"
 		(exclude_from_sim no)
@@
 	)
 	(junction
-		(at 63.5 34.29)
-		(diameter 0)
-		(color 0 0 0 0)
-	)
-	(junction
 		(at 248.92 69.85)
 		(diameter 0)
@@
 	)
 	(junction
+		(at 93.98 26.67)
+		(diameter 0)
+		(color 0 0 0 0)
+	)
+	(junction
 		(at 190.5 26.67)
 		(diameter 0)
@@
 	)
 	(no_connect
+		(at 63.5 58.42)
+	)
+	(no_connect
 		(at 182.88 242.57)
 	)
@@
 	)
 	(no_connect
-		(at 100.33 52.07)
-	)
-	(no_connect
 		(at 154.94 234.95)
 	)
@@
 	)
 	(no_connect
-		(at 100.33 49.53)
-	)
-	(no_connect
 		(at 182.88 224.79)
 	)
@@
 	(wire
 		(pts
-			(xy 90.17 26.67) (xy 102.87 26.67)
+			(xy 90.17 26.67) (xy 93.98 26.67)
 		)
 		(stroke
@@
 	(wire
 		(pts
-			(xy 48.26 34.29) (xy 63.5 34.29)
+			(xy 48.26 34.29) (xy 80.01 34.29)
 		)
 		(stroke
@@
 	(wire
 		(pts
-			(xy 63.5 58.42) (xy 63.5 34.29)
-		)
-		(stroke
-			(width 0.5)
-			(type default)
-		)
-	)
-	(wire
-		(pts
 			(xy 44.45 236.22) (xy 44.45 241.3)
 		)
@@
 	(wire
 		(pts
-			(xy 63.5 34.29) (xy 62.23 34.29)
-		)
-		(stroke
-			(width 0)
-			(type default)
-		)
-	)
-	(wire
-		(pts
 			(xy 133.35 35.56) (xy 133.35 38.1)
 		)
@@
 	(wire
 		(pts
+			(xy 93.98 26.67) (xy 102.87 26.67)
+		)
+		(stroke
+			(width 0.5)
+			(type default)
+		)
+	)
+	(wire
+		(pts
 			(xy 344.17 153.67) (xy 349.25 153.67)
 		)
@@
 	(wire
 		(pts
-			(xy 63.5 34.29) (xy 80.01 34.29)
-		)
-		(stroke
-			(width 0.5)
-			(type default)
-		)
-	)
-	(wire
-		(pts
 			(xy 298.45 195.58) (xy 340.36 195.58)
 		)
@@
 		)
 	)
+	(global_label "I2C0_SCL"
+		(shape input)
+		(at 100.33 52.07 0)
+		(fields_autoplaced yes)
+		(effects
+			(font
+				(size 1.27 1.27)
+			)
+			(justify left)
+		)
+		(property "Intersheetrefs" "${INTERSHEET_REFS}"
+			(at 112.0842 52.07 0)
+			(effects
+				(font
+					(size 1.27 1.27)
+				)
+				(justify left)
+				(hide yes)
+			)
+		)
+	)
 	(global_label "RTS"
 		(shape input)
@@
 		)
 	)
+	(global_label "I2C0_SDA"
+		(shape input)
+		(at 100.33 49.53 0)
+		(fields_autoplaced yes)
+		(effects
+			(font
+				(size 1.27 1.27)
+			)
+			(justify left)
+		)
+		(property "Intersheetrefs" "${INTERSHEET_REFS}"
+			(at 112.1447 49.53 0)
+			(effects
+				(font
+					(size 1.27 1.27)
+				)
+				(justify left)
+				(hide yes)
+			)
+		)
+	)
 	(global_label "BTN_2"
 		(shape input)
@@
 			)
 		)
-		(property "Value" "4.7k"
+		(property "Value" "1.3k"
 			(at 278.384 130.556 0)
 			(effects
@@
 			)
 		)
-		(property "LCSC PN" "C25900"
+		(property "LCSC PN" "C881388"
 			(at 276.86 129.54 0)
 			(effects
@@
 	)
 	(symbol
+		(lib_id "power:GNDPWR")
+		(at 93.98 19.05 180)
+		(unit 1)
+		(exclude_from_sim no)
+		(in_bom yes)
+		(on_board yes)
+		(dnp no)
+		(fields_autoplaced yes)
+		(property "Reference" "#PWR089"
+			(at 93.98 13.97 0)
+			(effects
+				(font
+					(size 1.27 1.27)
+				)
+				(hide yes)
+			)
+		)
+		(property "Value" "PGND1"
+			(at 94.107 15.24 0)
+			(effects
+				(font
+					(size 1.27 1.27)
+				)
+			)
+		)
+		(property "Footprint" ""
+			(at 93.98 17.78 0)
+			(effects
+				(font
+					(size 1.27 1.27)
+				)
+				(hide yes)
+			)
+		)
+		(property "Datasheet" ""
+			(at 93.98 17.78 0)
+			(effects
+				(font
+					(size 1.27 1.27)
+				)
+				(hide yes)
+			)
+		)
+		(property "Description" "Power symbol creates a global label with name \"GNDPWR\" , global ground"
+			(at 93.98 19.05 0)
+			(effects
+				(font
+					(size 1.27 1.27)
+				)
+				(hide yes)
+			)
+		)
+		(pin "1"
+		)
+		(instances
+			(project "main_board"
+				(path "/62950e93-3f98-4dee-9256-8213caa98ee7"
+					(reference "#PWR089")
+					(unit 1)
+				)
+			)
+		)
+	)
+	(symbol
 		(lib_id "Interface_USB:HUSB238_xxxDD")
 		(at 90.17 52.07 0)
@@
 	(symbol
 		(lib_id "Johnson_Symbol_Lib:PMOS_STL6P3LLH6")
-		(at 111.76 29.21 90)
+		(at 111.76 29.21 270)
+		(mirror x)
 		(unit 1)
 		(exclude_from_sim no)
@@
 		(on_board yes)
 		(dnp no)
-		(fields_autoplaced yes)
 		(property "Reference" "Q1"
 			(at 111.76 20.32 90)
@@
 		)
 		(property "Footprint" "Package_SON:VSON-8_3.3x3.3mm_P0.65mm_NexFET"
-			(at 109.22 24.13 0)
+			(at 114.3 24.13 0)
 			(effects
 				(font
@@
 			)
 		)
-		(property "Value" "10k"
+		(property "Value" "0"
 			(at 110.49 62.2299 0)
 			(effects
@@
 			)
 		)
-		(property "LCSC PN" "C25744"
+		(property "LCSC PN" "C17168"
 			(at 113.03 60.96 90)
 			(effects
@@
 	)
 	(symbol
+		(lib_id "Diode:SMF28A")
+		(at 93.98 22.86 90)
+		(unit 1)
+		(exclude_from_sim no)
+		(in_bom yes)
+		(on_board yes)
+		(dnp no)
+		(fields_autoplaced yes)
+		(property "Reference" "D5"
+			(at 96.52 21.5899 90)
+			(effects
+				(font
+					(size 1.27 1.27)
+				)
+				(justify right)
+			)
+		)
+		(property "Value" "SMF28A"
+			(at 96.52 24.1299 90)
+			(effects
+				(font
+					(size 1.27 1.27)
+				)
+				(justify right)
+			)
+		)
+		(property "Footprint" "Diode_SMD:D_SMF"
+			(at 99.06 22.86 0)
+			(effects
+				(font
+					(size 1.27 1.27)
+				)
+				(hide yes)
+			)
+		)
+		(property "Datasheet" "https://www.vishay.com/doc?85881"
+			(at 93.98 24.13 0)
+			(effects
+				(font
+					(size 1.27 1.27)
+				)
+				(hide yes)
+			)
+		)
+		(property "Description" "200W unidirectional Transil Transient Voltage Suppressor, 28Vrwm, SMF"
+			(at 93.98 22.86 0)
+			(effects
+				(font
+					(size 1.27 1.27)
+				)
+				(hide yes)
+			)
+		)
+		(pin "1"
+		)
+		(pin "2"
+		)
+		(instances
+			(project ""
+				(path "/62950e93-3f98-4dee-9256-8213caa98ee7"
+					(reference "D5")
+					(unit 1)
+				)
+			)
+		)
+	)
+	(symbol
 		(lib_id "Device:R_Small")
 		(at 265.43 38.1 0)
@@
 			)
 		)
-		(property "Value" "+5V"
+		(property "Value" "+3V3"
 			(at 358.14 31.496 0)
 			(effects
@@
 			)
 		)
-		(property "Value" "4.7k"
+		(property "Value" "1.3k"
 			(at 265.176 152.146 0)
 			(effects
@@
 			)
 		)
-		(property "Value" "4.7k"
+		(property "Value" "1.3k"
 			(at 270.256 152.4 0)
 			(effects
@@
 			)
 		)
-		(property "Value" "4.7k"
+		(property "Value" "1.3k"
 			(at 272.796 130.556 0)
 			(effects
@@
 			)
 		)
-		(property "LCSC PN" "C25900"
+		(property "LCSC PN" "C881388"
 			(at 274.32 129.54 0)
 			(effects
